Commit message: [P4-control][Agent B] Fix Holon battery inertial data

File: assets/robots/holon/holon.urdf (robot description, URDF)
Before this commit: robot holon, 29 links, 28 joints
Links:
- link battery2: mass 0 -> 0.208516276418653

File: module_urdf/holon.urdf.xacro (robot description, xacro)
@@ -704,7 +704,7 @@
   <link name="battery2">
     <inertial>
-      <origin xyz="0 0 0" rpy="0 0 0" />
-      <mass value="0" />
-      <inertia ixx="0" ixy="0" ixz="0" iyy="0" iyz="0" izz="0" />
+      <origin xyz="-5.98493495209129E-05 2.87169107937579E-11 -0.032069808029366" rpy="0 0 0" />
+      <mass value="0.208516276418653" />
+      <inertia ixx="0.000101484961957605" ixy="1.83742309473515E-13" ixz="-4.60685696556113E-07" iyy="0.000171408361564041" iyz="1.41515083699141E-13" izz="0.000132682759440689" />
     </inertial>
     <visual>

Commit message: [P4-full][Order0] Add joint actuator performance model

File: assets/robots/holon/holon.urdf (robot description, URDF)
Before this commit: robot holon, 29 links, 28 joints
Joints:
- joint gimbal1: limit lower=-2.0 upper=2.0 effort=6.6 velocity=3.0 -> lower=-2.0 upper=2.0 effort=0.76 velocity=10.890854
- joint gimbal2: limit lower=-2.0 upper=2.0 effort=6.6 velocity=3.0 -> lower=-2.0 upper=2.0 effort=0.76 velocity=10.890854
- joint gimbal3: limit lower=-2.0 upper=2.0 effort=6.6 velocity=3.0 -> lower=-2.0 upper=2.0 effort=0.76 velocity=10.890854
- joint gimbal4: limit lower=-2.0 upper=2.0 effort=6.6 velocity=3.0 -> lower=-2.0 upper=2.0 effort=0.76 velocity=10.890854
- joint pitch_dock_mech_joint1: limit lower=-1.5708 upper=1.5708 effort=6.6 velocity=3.0 -> lower=-1.5708 upper=1.5708 effort=4.1 velocity=45.553093
- joint pitch_dock_mech_joint2: limit lower=-1.5708 upper=1.5708 effort=6.6 velocity=3.0 -> lower=-1.5708 upper=1.5708 effort=4.1 velocity=45.553093
- joint yaw_dock_mech_joint1: limit lower=-1.5708 upper=1.5708 effort=6.6 velocity=3.0 -> lower=-1.5708 upper=1.5708 effort=4.1 velocity=45.553093
- joint yaw_dock_mech_joint2: limit lower=-1.5708 upper=1.5708 effort=6.6 velocity=3.0 -> lower=-1.5708 upper=1.5708 effort=4.1 velocity=45.553093

File: module_urdf/holon.urdf.xacro (robot description, xacro)
@@ -104,5 +104,5 @@
     <child link="gimbal_link1" />
     <axis xyz="1 0 0" />
-    <limit lower="-2.0" upper="2.0" effort="6.6" velocity="3.0" />
+    <limit lower="-2.0" upper="2.0" effort="0.76" velocity="10.890854" />
     <dynamics damping="0.8" friction="0.0" />
   </joint>
@@ -185,5 +185,5 @@
     <child link="pitch_dock_mech1" />
     <axis xyz="0 1 0" />
-    <limit lower="-1.5708" upper="1.5708" effort="6.6" velocity="3.0" />
+    <limit lower="-1.5708" upper="1.5708" effort="4.1" velocity="45.553093" />
     <dynamics damping="0.8" friction="0.0" />
   </joint>
@@ -257,5 +257,5 @@
     <child link="gimbal_link2" />
     <axis xyz="1 0 0" />
-    <limit lower="-2.0" upper="2.0" effort="6.6" velocity="3.0" />
+    <limit lower="-2.0" upper="2.0" effort="0.76" velocity="10.890854" />
     <dynamics damping="0.8" friction="0.0" />
   </joint>
@@ -346,5 +346,5 @@
     <child link="yaw_dock_mech1" />
     <axis xyz="0 0 1" />
-    <limit lower="-1.5708" upper="1.5708" effort="6.6" velocity="3.0" />
+    <limit lower="-1.5708" upper="1.5708" effort="4.1" velocity="45.553093" />
     <dynamics damping="0.8" friction="0.0" />
   </joint>
@@ -410,5 +410,5 @@
     <child link="gimbal_link3" />
     <axis xyz="1 0 0" />
-    <limit lower="-2.0" upper="2.0" effort="6.6" velocity="3.0" />
+    <limit lower="-2.0" upper="2.0" effort="0.76" velocity="10.890854" />
     <dynamics damping="0.8" friction="0.0" />
   </joint>
@@ -491,5 +491,5 @@
     <child link="yaw_dock_mech2" />
     <axis xyz="0 0 1" />
-    <limit lower="-1.5708" upper="1.5708" effort="6.6" velocity="3.0" />
+    <limit lower="-1.5708" upper="1.5708" effort="4.1" velocity="45.553093" />
     <dynamics damping="0.8" friction="0.0" />
   </joint>
@@ -563,5 +563,5 @@
     <child link="gimbal_link4" />
     <axis xyz="1 0 0" />
-    <limit lower="-2.0" upper="2.0" effort="6.6" velocity="3.0" />
+    <limit lower="-2.0" upper="2.0" effort="0.76" velocity="10.890854" />
     <dynamics damping="0.8" friction="0.0" />
   </joint>
@@ -652,5 +652,5 @@
     <child link="pitch_dock_mech2" />
     <axis xyz="0 1 0" />
-    <limit lower="-1.5708" upper="1.5708" effort="6.6" velocity="3.0" />
+    <limit lower="-1.5708" upper="1.5708" effort="4.1" velocity="45.553093" />
     <dynamics damping="0.8" friction="0.0" />
   </joint>

Commit message: [P4-full][Order3] Integrate Isaac rollout pipeline

File: assets/robots/holon/holon.urdf (robot description, URDF)
Before this commit: robot holon, 29 links, 28 joints
Joints:
- joint pitch_dock_mech_joint2: origin xyz=0.145 0 0 rpy=0 0.031857 0 -> xyz=0.145 0 0 rpy=0 0 0
- joint yaw_dock_mech_joint1: origin xyz=0.145 0 0 rpy=0 0 0.006433 -> xyz=0.145 0 0 rpy=0 0 0
- joint yaw_dock_mech_joint2: origin xyz=0.145 0 0 rpy=0 0 0.021103 -> xyz=0.145 0 0 rpy=0 0 0

File: module_urdf/holon.urdf.xacro (robot description, xacro)
@@ -342,5 +342,5 @@
   </gazebo>
   <joint name="yaw_dock_mech_joint1" type="revolute">
-    <origin xyz="0.145 0 0" rpy="0 0 0.006433" />
+    <origin xyz="0.145 0 0" rpy="0 0 0" />
     <parent link="rotor_arm2" />
     <child link="yaw_dock_mech1" />
@@ -487,5 +487,5 @@
   </gazebo>
   <joint name="yaw_dock_mech_joint2" type="revolute">
-    <origin xyz="0.145 0 0" rpy="0 0 0.021103" />
+    <origin xyz="0.145 0 0" rpy="0 0 0" />
     <parent link="rotor_arm3" />
     <child link="yaw_dock_mech2" />
@@ -648,5 +648,5 @@
   </gazebo>
   <joint name="pitch_dock_mech_joint2" type="revolute">
-    <origin xyz="0.145 0 0" rpy="0 0.031857 0" />
+    <origin xyz="0.145 0 0" rpy="0 0 0" />
     <parent link="rotor_arm4" />
     <child link="pitch_dock_mech2" />

Commit message: [P4-full][Order9] Build collision-safe C3 nominal trajectories

File: assets/robots/holon/holon.urdf (robot description, URDF)
Before this commit: robot holon, 29 links, 28 joints
Links:
- added link pitch_grasp_contact_frame_1
- added link pitch_grasp_contact_frame_2
- link rotor_arm1: geometry collision mesh filename=mesh/rotor_arm_pitch.STL; visual mesh filename=mesh/rotor_arm_pitch.STL
- link rotor_arm4: geometry collision mesh filename=mesh/rotor_arm_pitch.STL; visual mesh filename=mesh/rotor_arm_pitch.STL
Joints:
- added joint pitch_grasp_contact_frame_joint_1: type fixed, parent pitch_connect_dummy_1, child pitch_grasp_contact_frame_1, origin xyz=0.0424086 0 0 rpy=0 0 0
- added joint pitch_grasp_contact_frame_joint_2: type fixed, parent pitch_connect_dummy_2, child pitch_grasp_contact_frame_2, origin xyz=0.0424086 0 0 rpy=0 0 0

File: module_urdf/holon.urdf.xacro (robot description, xacro)
@@ -61,5 +61,5 @@
       <origin xyz="0 0 0" rpy="0 0 0" />
       <geometry>
-        <mesh filename="mesh/rotor_arm_1.STL" />
+        <mesh filename="mesh/rotor_arm_pitch.STL" />
       </geometry>
     </collision>
@@ -162,5 +162,5 @@
     </inertial>
     <visual>
-      <origin xyz="0 0 0" rpy="0 0 1.5708" />
+      <origin xyz="0 0 0" rpy="3.14159265358979 0 0" />
       <geometry>
         <mesh filename="mesh/pitch_dock_mech_1.STL" />
@@ -171,5 +171,5 @@
     </visual>
     <collision>
-      <origin xyz="0 0 0" rpy="0 0 1.5708" />
+      <origin xyz="0 0 0" rpy="3.14159265358979 0 0" />
       <geometry>
         <mesh filename="mesh/pitch_dock_mech_1.STL" />
@@ -196,4 +196,11 @@
     <axis xyz="0 1 0" />
   </joint>
+  <link name="pitch_grasp_contact_frame_1">
+  </link>
+  <joint name="pitch_grasp_contact_frame_joint_1" type="fixed">
+    <origin xyz="0.0424086 0 0" rpy="0 0 0" />
+    <parent link="pitch_connect_dummy_1" />
+    <child link="pitch_grasp_contact_frame_1" />
+  </joint>
   <link name="rotor_arm2">
     <inertial>
@@ -520,5 +527,5 @@
       <origin xyz="0 0 0" rpy="0 0 0" />
       <geometry>
-        <mesh filename="mesh/rotor_arm_4.STL" />
+        <mesh filename="mesh/rotor_arm_pitch.STL" />
       </geometry>
     </collision>
@@ -621,5 +628,5 @@
     </inertial>
     <visual>
-      <origin xyz="0 0 0" rpy="0 0 1.5708" />
+      <origin xyz="0 0 0" rpy="3.14159265358979 0 0" />
       <geometry>
         <mesh filename="mesh/pitch_dock_mech_2.STL" />
@@ -630,5 +637,5 @@
     </visual>
     <collision>
-      <origin xyz="0 0 0" rpy="0 0 1.5708" />
+      <origin xyz="0 0 0" rpy="3.14159265358979 0 0" />
       <geometry>
         <mesh filename="mesh/pitch_dock_mech_2.STL" />
@@ -643,4 +650,11 @@
     <child link="pitch_connect_dummy_2" />
     <axis xyz="0 1 0" />
+  </joint>
+  <link name="pitch_grasp_contact_frame_2">
+  </link>
+  <joint name="pitch_grasp_contact_frame_joint_2" type="fixed">
+    <origin xyz="0.0424086 0 0" rpy="0 0 0" />
+    <parent link="pitch_connect_dummy_2" />
+    <child link="pitch_grasp_contact_frame_2" />
   </joint>
   <gazebo reference="pitch_dock_mech2">
